File: pcb/omni-wheel/omni-wheel.kicad_sch (KiCad schematic)
At the start: 4 parts, among them J1 Motor1_input, J2 Motor_2input, J3 Motor1_input, J4 Motor1_input

Commit message: Working on Circuit design, got major components down schematic
Parts:
- added C1: .1uF, symbol Device:C
- added C2: .1 uF, symbol Device:C
- added J5: STLINK, symbol Connector:Conn_01x04_Socket
- added J6: 3.3V Input, symbol Connector_Generic:Conn_01x02
- added J7: 12V Input, symbol Connector_Generic:Conn_01x02
- added U1, U2: SN754410NE, Package_DIP:DIP-16_W7.62mm, symbol Driver_Motor:SN754410NE
- added U3: STM32F030R8Tx, Package_QFP:LQFP-64_10x10mm_P0.5mm, symbol MCU_ST_STM32F0:STM32F030R8Tx
- J2: value Motor_2input -> Motor2_input
- J3: value Motor1_input -> Motor4_input
- J4: value Motor1_input -> Motor3_input
Connections:
- net +3.3V: now also C1.2, J6.1 (Pin_1), U3.32 (VDD)
- net GND: now also C1.1, C2.1, J5.4 (Pin_4), J6.2 (Pin_2), J7.2 (Pin_2), U1.12 (GND), U1.13 (GND), U1.4 (GND), U1.5 (GND), U2.12 (GND), U2.13 (GND), U2.4 (GND), U2.5 (GND), U3.31 (VSS), U3.63 (VSS)
- removed net ENC_A: J1.3 (Pin_3), J2.3 (Pin_3), J3.3 (Pin_3), J4.3 (Pin_3)
- removed net ENC_B: J1.4 (Pin_4), J2.4 (Pin_4), J3.4 (Pin_4), J4.4 (Pin_4)
- removed net M1: J1.1 (Pin_1), J2.1 (Pin_1), J3.1 (Pin_1), J4.1 (Pin_1)
- removed net M2: J1.6 (Pin_6), J2.6 (Pin_6), J3.6 (Pin_6), J4.6 (Pin_6)
- new net: J5.3 (Pin_3), U3.46 (PA13)
- new net: J5.2 (Pin_2), U3.49 (PA14)
- new net: C2.2, J5.1 (Pin_1), U3.64 (VDD)
- new net +12V: J7.1 (Pin_1), U1.16 (VCC1), U1.8 (VCC2), U2.16 (VCC1), U2.8 (VCC2)
- new net Motor1_ENC_A: J1.3 (Pin_3)
- new net Motor1_ENC_B: J1.4 (Pin_4)
- new net Motor1_M1: J1.1 (Pin_1), U1.3 (1Y)
- new net Motor1_M2: J1.6 (Pin_6), U1.6 (2Y)
- new net Motor2_ENC_A: J2.3 (Pin_3)
- new net Motor2_ENC_B: J2.4 (Pin_4)
- new net Motor2_M1: J2.1 (Pin_1), U1.11 (3Y)
- new net Motor2_M2: J2.6 (Pin_6), U1.14 (4Y)
- new net Motor3_ENC_A: J4.3 (Pin_3)
- new net Motor3_ENC_B: J4.4 (Pin_4)
- new net Motor3_M1: J4.1 (Pin_1), U2.3 (1Y)
- new net Motor3_M2: J4.6 (Pin_6), U2.6 (2Y)
- new net Motor4_ENC_A: J3.3 (Pin_3)
- new net Motor4_ENC_B: J3.4 (Pin_4)
- new net Motor4_M1: J3.1 (Pin_1), U2.11 (3Y)
- new net Motor4_M2: J3.6 (Pin_6), U2.14 (4Y)
Other:
- moved on the sheet: J1, J2
