File: pcb/omni-wheel/omni-wheel.kicad_pcb (KiCad board)
At the start: 2 copper layers, 3 parts, among them U1 SN754410NE, U2 SN754410NE, U3 STM32F030R8Tx

Commit message: PCB save
Parts:
- added U4: SN74HCT74DR, SN74HCT74DR:D14, F.Cu at (220.5, 81.5)
- added U5: SN74HCT74DR, SN74HCT74DR:D14, F.Cu at (256.0, 82.2)
- moved U2 153.4 mm to (275.5, 96.0), turned to 180 degrees
- moved U3 109.6 mm to (239.8, 85.8)
- moved U1 94.9 mm to (204.0, 97.0), turned to 180 degrees

Commit message: pcb update for home
Parts:
- added J6: 3.3V Input, Connector_AMASS:AMASS_XT60PW-M_1x02_P7.20mm_Horizontal, F.Cu at (273.9, 120.5)
- added J7: 12V Input, Connector_AMASS:AMASS_XT60PW-M_1x02_P7.20mm_Horizontal, F.Cu at (199.6, 120.5)
- added J8: 5V Input, Connector_AMASS:AMASS_XT60PW-M_1x02_P7.20mm_Horizontal, F.Cu at (251.6, 120.8)
- added U6: SN74AC86DR, SN74AC86DR:D14, F.Cu at (236.7, 102.5)
- moved U5 11.8 mm to (250.5, 71.8)
- moved U4 11.1 mm to (221.5, 70.5)
- moved U1 2.88 mm to (201.1, 97.0)
- moved U2 2.88 mm to (272.6, 96.0)
- moved U3 2.88 mm to (236.9, 85.8)
Connections:
- net /Motor1_ENCB renamed /Motor1_Dir
- net /Motor2_ENCB renamed /Motor2_Dir
- net /Motor3_ENCB renamed /Motor3_Dir
- net /Motor4_ENCB renamed /Motor4_Dir
- U3 pad 10: /Motor1_ENCA -> /Motor1_EncTicks
- U3 pad 3: /Motor4_ENCA -> /Motor4_EncTicks
- U3 pad 37: /Motor2_ENCA -> /Motor2_EncTicks
- U3 pad 51: /Motor3_ENCA -> /Motor3_EncTicks

Commit message: power distribution done, lay up  is next
Parts:
- removed U5: SN74HCT74DR, SN74HCT74DR:D14
- added C1: .1 uF, Capacitor_SMD:C_0603_1608Metric, F.Cu at (222.8, 65.5)
- added C11: 10uF, Capacitor_SMD:C_0603_1608Metric, F.Cu at (218.2, 58.5)
- added C12: 100nF, Capacitor_SMD:C_0603_1608Metric, F.Cu at (218.2, 61.0)
- added C2: .1 uF, Capacitor_SMD:C_0603_1608Metric, F.Cu at (222.8, 68.0)
- added C3: 100nF, Capacitor_SMD:C_0603_1608Metric, F.Cu at (214.2, 56.0)
- added C4: 47pF, Capacitor_SMD:C_0603_1608Metric, F.Cu at (214.2, 58.5)
- added C5: 22uF, Capacitor_SMD:C_0603_1608Metric, F.Cu at (214.2, 61.0)
- added C6: 22uF, Capacitor_SMD:C_0603_1608Metric, F.Cu at (214.2, 63.5)
- added C7: 22uF, Capacitor_SMD:C_0603_1608Metric, F.Cu at (214.2, 66.0)
- added C8: 22uF, Capacitor_SMD:C_0603_1608Metric, F.Cu at (214.2, 68.5)
- added C9: 56pF, Capacitor_SMD:C_0603_1608Metric, F.Cu at (218.2, 56.0)
- added J1: Motor1_output, Connector_JST:JST_PH_B6B-PH-K_1x06_P2.00mm_Vertical, F.Cu at (157.2, 90.5)
- added J2: Motor2_output, Connector_JST:JST_PH_B6B-PH-K_1x06_P2.00mm_Vertical, F.Cu at (188.7, 115.5)
- added J3: Motor4_output, Connector_JST:JST_PH_B6B-PH-K_1x06_P2.00mm_Vertical, F.Cu at (226.5, 89.5)
- added J4: Motor3_output, Connector_JST:JST_PH_B6B-PH-K_1x06_P2.00mm_Vertical, F.Cu at (192.5, 54.5)
- added L1: 6.8u, Inductor_SMD:L_0603_1608Metric, F.Cu at (218.2, 63.5)
- added L2: 4.7u, Inductor_SMD:L_0603_1608Metric, F.Cu at (218.2, 66.0)
- added R1: 158k, Resistor_SMD:R_0603_1608Metric, F.Cu at (218.2, 68.5)
- added R2: 30.1k, Resistor_SMD:R_0603_1608Metric, F.Cu at (222.2, 56.0)
- added R3: 93.1k, Resistor_SMD:R_0603_1608Metric, F.Cu at (222.2, 58.5)
- added R4: 30.1k, Resistor_SMD:R_0603_1608Metric, F.Cu at (222.2, 61.0)
- J6, J8: footprint Connector_AMASS:AMASS_XT60PW-M_1x02_P7.20mm_Horizontal -> Connector_AMASS:AMASS_XT30PW-M_1x02_P2.50mm_Horizontal
- U4: value SN74HCT74DR -> CD74HC04E; footprint SN74HCT74DR:D14 -> CD74HC04E:N14
- moved J8 81.0 mm to (171.0, 113.3)
- moved U2 77.4 mm to (199.6, 70.4), turned to -90 degrees
- moved J6 64.7 mm to (209.5, 113.8)
- moved J7 64.5 mm to (164.2, 66.6), turned to 90 degrees
- moved U6 33.6 mm to (211.7, 80.0)
- moved U4 27.5 mm to (197.5, 83.9), turned to 90 degrees
- moved U3 27.4 mm to (211.5, 96.0)
- moved U1 2.52 mm to (198.7, 96.4), turned to -90 degrees
Connections:
- U3 pad 11: /Motor1_Dir -> unconnected-(U3-PC3-Pad11)
- U3 pad 2: /Motor4_4A -> /Motor4_EN
- U3 pad 25: /Motor2_4A -> /Motor2_EN
- U3 pad 38: /Motor2_Dir -> unconnected-(U3-PC7-Pad38)
- U3 pad 4: /Motor4_Dir -> unconnected-(U3-PC15-Pad4)
- U3 pad 40: /Motor3_2A -> /Motor3_EN
- U3 pad 52: /Motor3_Dir -> unconnected-(U3-PC11-Pad52)
- U3 pad 9: /Motor1_2A -> /Motor1_EN
- U4 pad 1: unconnected-(U4-*1CLR-Pad1) -> /Motor1_1A
- U4 pad 14: unconnected-(U4-VCC-Pad14) -> +5V
- U4 pad 2: unconnected-(U4-1D-Pad2) -> /Motor1_2A
- U4 pad 3: unconnected-(U4-1CLK-Pad3) -> /Motor2_3A
- U4 pad 4: unconnected-(U4-*1PRE-Pad4) -> /Motor2_4A
- U4 pad 5: unconnected-(U4-1Q-Pad5) -> /Motor3_1A
- U4 pad 6: unconnected-(U4-*1Q-Pad6) -> /Motor3_2A
- U4 pad 7: unconnected-(U4-GND-Pad7) -> GND
- U4 pad 8: unconnected-(U4-*2Q-Pad8) -> /Motor4_4A
- U4 pad 9: unconnected-(U4-2Q-Pad9) -> /Motor4_3A

Commit message: pcb update for home
Parts:
- removed J1: Motor1_output, Connector_JST:JST_PH_B6B-PH-K_1x06_P2.00mm_Vertical
- removed J8: 5V Input, Connector_AMASS:AMASS_XT30PW-M_1x02_P2.50mm_Horizontal
- added IC1: AP63301WU-7, footprints:SOT95P280X100-6N, F.Cu at (83.8, 58.5)
- added IC2: AP63301WU-7, footprints:SOT95P280X100-6N, F.Cu at (83.8, 70.0)
- added REF**: MountingHole_2.2mm_M2, MountingHole:MountingHole_2.2mm_M2, F.Cu at (126.5, 51.0)
- added REF**: MountingHole_2.2mm_M2, MountingHole:MountingHole_2.2mm_M2, F.Cu at (126.5, 104.5)
- added REF**: MountingHole_2.2mm_M2, MountingHole:MountingHole_2.2mm_M2, F.Cu at (73.5, 104.5)
- added REF**: MountingHole_2.2mm_M2, MountingHole:MountingHole_2.2mm_M2, F.Cu at (73.5, 50.5)
- J6: value 3.3V Input -> Motor1_output; footprint Connector_AMASS:AMASS_XT30PW-M_1x02_P2.50mm_Horizontal -> Connector_JST:JST_PH_B6B-PH-K_1x06_P2.00mm_Vertical
- moved R3 181.6 mm to (41.2, 73.0)
- moved R4 181.6 mm to (41.2, 75.5)
- moved C1 181.6 mm to (41.8, 80.0)
- moved C12 181.6 mm to (37.2, 75.5)
- moved C2 181.6 mm to (41.8, 82.5)
- moved L2 181.6 mm to (37.2, 80.5)
- moved C11 181.0 mm to (37.3, 55.0)
- moved C9 173.8 mm to (44.5, 59.5)
- moved C5 153.7 mm to (62.8, 34.5)
- moved C6 153.7 mm to (62.8, 37.0)
- moved C7 153.7 mm to (62.8, 39.5)
- moved C8 153.7 mm to (62.8, 42.0)
- moved J6 140.0 mm to (75.0, 75.0), turned to -90 degrees
- moved L1 127.8 mm to (90.5, 58.2), turned to -90 degrees
- moved C3 126.7 mm to (87.5, 58.2), turned to 90 degrees
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Connections:
- J6 pad 1: +3.3V -> /Motor1_M1
Routing:
- net /Motor2_ENCA: track 0.00 -> 29.5 mm
- net /Motor2_ENCB: track 0.00 -> 29.0 mm
- net /Motor3_ENCB: track 0.00 -> 28.2 mm
- net /Motor3_ENCA: track 0.00 -> 27.8 mm
- net /Motor1_ENCB: track 0.00 -> 22.4 mm
- net /Motor1_ENCA: track 0.00 -> 21.0 mm
- net /Motor4_ENCA: track 0.00 -> 18.8 mm
- net Net-(IC1-FB): track 0.00 -> 18.7 mm
- net /Motor4_ENCB: track 0.00 -> 17.4 mm
- net +12V: track 0.00 -> 10.4 mm
- net +5V: track 0.00 -> 6.04 mm
- net Net-(IC1-SW): track 0.00 -> 5.63 mm
- net Net-(IC1-BST): track 0.00 -> 2.42 mm
- added copper zone on B.Cu, net GND
Other:
- board outline added: 60 x 60 mm

Commit message: routing almost done, need to logic pins next
Parts:
- moved C1 63.5 mm to (105.0, 74.5), turned to 45 degrees
- moved R4 58.5 mm to (98.0, 61.3), turned to -90 degrees
- moved R3 54.2 mm to (94.5, 63.3), turned to 90 degrees
- moved L2 54.1 mm to (89.5, 66.5), turned to 90 degrees
- moved C12 53.7 mm to (89.5, 63.3), turned to 90 degrees
- moved C9 47.2 mm to (91.5, 63.3), turned to 90 degrees
- moved C11 46.4 mm to (81.0, 70.5), turned to -90 degrees
- moved C5 30.9 mm to (87.5, 53.0), turned to 180 degrees
- moved C7 30.8 mm to (90.5, 53.0), turned to 180 degrees
- moved C8 29.3 mm to (90.5, 51.5)
- moved C6 28.7 mm to (87.5, 51.5)
- moved C2 7.55 mm to (34.3, 83.5)
- moved IC2 6.61 mm to (85.0, 63.5)
- moved U3 2.85 mm to (109.5, 81.5), turned to -45 degrees
Connections:
- IC1 pad 4: unconnected-(IC1-GND-Pad4) -> GND
- IC2 pad 4: unconnected-(IC2-GND-Pad4) -> GND
- L2 pad 2: unconnected-(L2-Pad2) -> Net-(IC2-SW)
- U1 pad 16: +12V -> +5V
- U2 pad 16: +12V -> +5V
Routing:
- net +3.3V: track 0.00 -> 113.8 mm, vias 0 -> 2
- net /Motor4_M2: track 0.00 -> 24.5 mm
- net /Motor2_M2: track 0.00 -> 19.1 mm, vias 0 -> 2
- net /Motor1_M1: track 0.00 -> 19.1 mm, vias 0 -> 2
- net +12V: track 10.4 -> 25.6 mm
- net /Motor2_M1: track 0.00 -> 11.0 mm
- net Net-(IC2-FB): track 0.00 -> 10.8 mm
- net GND: track 0.00 -> 9.60 mm, vias 0 -> 5
- net /Motor1_M2: track 0.00 -> 9.49 mm
- net +5V: track 6.04 -> 12.3 mm
- net Net-(IC2-SW): track 0.00 -> 5.12 mm
- net Net-(IC2-BST): track 0.00 -> 3.51 mm
- net Net-(C7-Pad1): track 0.00 -> 1.50 mm
- net Net-(C5-Pad1): track 0.00 -> 1.50 mm

Commit message: save before architecture change
Parts:
- added C10: .1 uF, Capacitor_SMD:C_0603_1608Metric, F.Cu at (128.0, 110.0)
- added C13: .1 uF, Capacitor_SMD:C_0603_1608Metric, F.Cu at (148.2, 122.5)
- added C14: .1 uF, Capacitor_SMD:C_0603_1608Metric, F.Cu at (86.0, 111.0)
- added C15: .1 uF, Capacitor_SMD:C_0603_1608Metric, F.Cu at (103.7, 122.5)
- added C16: .1 uF, Capacitor_SMD:C_0603_1608Metric, F.Cu at (175.3, 56.5)
- added C17: .1 uF, Capacitor_SMD:C_0603_1608Metric, F.Cu at (173.2, 32.0)
- moved C2 148.5 mm to (171.0, 25.5), turned to 180 degrees
- moved REF** 86.5 mm to (159.5, 131.0)
- moved C1 86.3 mm to (175.7, 25.0), turned to 0 degrees
- moved REF** 79.0 mm to (73.5, 129.5)
- moved U1 65.5 mm to (145.6, 113.0), turned to -90 degrees
- moved J6 61.2 mm to (135.0, 87.0), turned to 90 degrees
- moved U2 59.1 mm to (84.8, 120.6), turned to 90 degrees
- moved REF** 56.8 mm to (97.5, 53.0)
- moved REF** 51.5 mm to (134.0, 53.5)
- moved J2 43.0 mm to (135.0, 108.5), turned to 90 degrees
- moved IC1 38.2 mm to (121.6, 64.3), turned to -90 degrees
- moved J7 37.3 mm to (112.7, 56.2), turned to 0 degrees
- moved C5 36.7 mm to (118.0, 73.3), turned to -90 degrees
- moved C6 36.3 mm to (116.5, 73.3), turned to 90 degrees
- moved C3 35.9 mm to (121.8, 68.8), turned to 0 degrees
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Connections:
- U3 pad 10: /Motor1_EncTicks -> /Motor2_3A
- U3 pad 11: unconnected-(U3-PC3-Pad11) -> /Motor1_1A
- U3 pad 16: /Motor1_EN -> unconnected-(U3-PA2-Pad16)
- U3 pad 2: /Motor4_EN -> unconnected-(U3-PC13-Pad2)
- U3 pad 20: /Motor2_EN -> unconnected-(U3-PA4-Pad20)
- U3 pad 22: /Motor3_EN -> unconnected-(U3-PA6-Pad22)
- U3 pad 23: /Motor4_EN -> unconnected-(U3-PA7-Pad23)
- U3 pad 24: /Motor2_3A -> unconnected-(U3-PC4-Pad24)
- U3 pad 25: /Motor2_EN -> unconnected-(U3-PC5-Pad25)
- U3 pad 3: /Motor4_EncTicks -> unconnected-(U3-PC14-Pad3)
- U3 pad 38: unconnected-(U3-PC7-Pad38) -> /Motor1_EncTicks
- U3 pad 39: /Motor3_1A -> /Motor4_EncTicks
- U3 pad 40: /Motor3_EN -> /Motor3_EncTicks
- U3 pad 50: unconnected-(U3-PA15-Pad50) -> /Motor1_EN
- U3 pad 51: /Motor3_EncTicks -> /Motor2_EN
- U3 pad 52: unconnected-(U3-PC11-Pad52) -> /Motor3_EN
- U3 pad 53: /Motor4_3A -> /Motor4_EN
- U3 pad 8: /Motor1_1A -> /Motor4_3A
- U3 pad 9: /Motor1_EN -> /Motor3_1A
- U4 pad 1: /Motor1_1A -> unconnected-(U4-1A-Pad1)
- U4 pad 10: unconnected-(U4-*5Y-Pad10) -> /Motor3_2A
- U4 pad 11: unconnected-(U4-5A-Pad11) -> /Motor3_1A
- U4 pad 2: /Motor1_2A -> unconnected-(U4-*1Y-Pad2)
- U4 pad 5: /Motor3_1A -> /Motor1_1A
- U4 pad 6: /Motor3_2A -> /Motor1_2A
- U6 pad 1: /Motor1_ENCA -> /Motor2_ENCA
- U6 pad 10: /Motor3_ENCB -> /Motor4_ENCB
- U6 pad 11: /Motor4_EncTicks -> /Motor3_EncTicks
- U6 pad 12: /Motor4_ENCA -> /Motor3_ENCA
- U6 pad 13: /Motor4_ENCB -> /Motor3_ENCB
- U6 pad 2: /Motor1_ENCB -> /Motor2_ENCB
- U6 pad 3: /Motor1_EncTicks -> /Motor2_EncTicks
- U6 pad 4: /Motor2_ENCA -> /Motor1_ENCA
- U6 pad 5: /Motor2_ENCB -> /Motor1_ENCB
- U6 pad 6: /Motor2_EncTicks -> /Motor1_EncTicks
- U6 pad 8: /Motor3_EncTicks -> /Motor4_EncTicks
- U6 pad 9: /Motor3_ENCA -> /Motor4_ENCA
Routing:
- net /Motor1_EN: track 0.00 -> 147.2 mm
- net +12V: track 25.6 -> 151.0 mm, vias 0 -> 2
- net /Motor2_EN: track 0.00 -> 107.5 mm, vias 0 -> 2
- net +5V: track 12.3 -> 119.5 mm, vias 0 -> 4
- net /Motor3_1A: track 0.00 -> 45.6 mm, vias 0 -> 1
- net /Motor3_EN: track 0.00 -> 44.6 mm, vias 0 -> 1
- net /Motor1_1A: track 0.00 -> 42.0 mm
- net /Motor1_M2: track 9.49 -> 51.3 mm
- net /Motor2_3A: track 0.00 -> 33.5 mm
- net /Motor2_4A: track 0.00 -> 26.0 mm
- net /Motor4_3A: track 0.00 -> 25.8 mm
- net /Motor4_4A: track 0.00 -> 25.6 mm
- net /Motor4_M2: track 24.5 -> 0.00 mm
- net /Motor2_M2: track 19.1 -> 0.00 mm, vias 2 -> 0
- net /Motor1_M1: track 19.1 -> 0.00 mm, vias 2 -> 0
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Other:
- board size 60 x 60 mm -> 92.5 x 92.5 mm
- board text added: "J6"

Commit message: save before architecture change
Parts:
- moved C10 91.6 mm to (219.6, 110.5)
- moved C13 91.6 mm to (239.8, 123.0)
- moved C14 91.6 mm to (177.6, 111.5)
- moved C15 91.6 mm to (195.3, 123.0)
- moved U1 91.6 mm to (237.2, 113.5)
- moved U2 91.6 mm to (176.4, 121.1)
- moved REF** 17.1 mm to (151.0, 52.0)
- moved REF** 17.0 mm to (80.5, 53.5)
- moved J4 8.45 mm to (98.5, 99.0)
- moved J3 7.68 mm to (98.5, 81.8)
- moved J6 7.01 mm to (131.5, 93.1)
- moved U4 4.38 mm to (111.4, 118.8)
- moved U6 4.38 mm to (115.5, 88.3)
- moved U3 4.38 mm to (114.8, 104.2)
- moved J2 3.54 mm to (131.5, 109.0)
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Routing:
- net +3.3V: track 131.2 -> 79.4 mm
- net +5V: track 119.5 -> 88.0 mm, vias 4 -> 3
- net +12V: track 151.0 -> 129.0 mm, vias 2 -> 1
- net /Motor2_ENCA: track 24.0 -> 42.6 mm
- net /Motor2_ENCB: track 23.7 -> 41.2 mm
- net /Motor4_ENCB: track 20.6 -> 35.0 mm
- net /Motor4_ENCA: track 20.7 -> 34.6 mm
- net /Motor3_ENCB: track 25.6 -> 38.2 mm
- net /Motor1_ENCA: track 17.5 -> 30.0 mm
- net /Motor3_ENCA: track 25.3 -> 36.7 mm
- net /Motor1_ENCB: track 17.8 -> 29.0 mm
- net /Motor3_1A: track 45.6 -> 38.6 mm
- net /Motor4_4A: track 25.6 -> 22.0 mm
- net /Motor1_2A: track 13.0 -> 9.58 mm
- net /Motor3_2A: track 12.3 -> 11.4 mm
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- added copper zone on F.Cu, net +12V
- added copper zone on F.Cu, net +3.3V
- added copper zone on F.Cu, net +5V
Other:
- board text added: "12V"
- board text added: "3.3V"
- board text added: "5V"

Commit message: first pcb revision done
Parts:
- moved C13 158.4 mm to (81.5, 117.0), turned to 90 degrees
- moved C10 118.2 mm to (102.7, 128.0), turned to 0 degrees
- moved C2 105.4 mm to (107.0, 109.2), turned to -90 degrees
- moved C16 102.6 mm to (109.2, 135.0), turned to -90 degrees
- moved U2 95.0 mm to (81.6, 127.8)
- moved C1 92.4 mm to (122.5, 100.5), turned to 90 degrees
- moved C17 87.0 mm to (113.0, 94.8), turned to -90 degrees
- moved U1 84.0 mm to (153.4, 118.7)
- moved C15 62.3 mm to (133.0, 122.8), turned to -90 degrees
- moved J7 36.9 mm to (147.9, 65.6), turned to -90 degrees
- moved C11 35.4 mm to (144.6, 62.7), turned to 90 degrees
- moved C14 30.1 mm to (153.2, 129.3), turned to -90 degrees
- moved IC2 28.3 mm to (139.8, 64.9), turned to 180 degrees
- moved C8 27.7 mm to (130.8, 59.9), turned to 0 degrees
- moved L2 27.7 mm to (135.3, 61.9), turned to -90 degrees
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Connections:
- U3 pad 16: unconnected-(U3-PA2-Pad16) -> /Motor2_EN
- U3 pad 20: unconnected-(U3-PA4-Pad20) -> /Motor1_EN
- U3 pad 22: unconnected-(U3-PA6-Pad22) -> /Motor4_EN
- U3 pad 23: unconnected-(U3-PA7-Pad23) -> /Motor3_EN
- U3 pad 50: /Motor1_EN -> unconnected-(U3-PA15-Pad50)
- U3 pad 51: /Motor2_EN -> unconnected-(U3-PC10-Pad51)
- U3 pad 52: /Motor3_EN -> unconnected-(U3-PC11-Pad52)
- U3 pad 53: /Motor4_EN -> unconnected-(U3-PC12-Pad53)
Routing:
- net +12V: track 129.0 -> 249.4 mm
- net +3.3V: track 79.4 -> 194.7 mm, vias 3 -> 2
- net /Motor1_EN: track 147.2 -> 38.0 mm
- net /Motor2_EN: track 107.5 -> 29.3 mm, vias 2 -> 1
- net +5V: track 88.0 -> 19.3 mm, vias 3 -> 0
- net /Motor2_M2: track 0.00 -> 62.3 mm, vias 0 -> 1
- net /Motor4_M1: track 0.00 -> 44.5 mm, vias 0 -> 1
- net /Motor2_M1: track 0.00 -> 40.0 mm, vias 0 -> 1
- net /Motor1_M1: track 0.00 -> 39.5 mm, vias 0 -> 1
- net /Motor3_M1: track 0.78 -> 39.9 mm, vias 0 -> 1
- net /Motor4_M2: track 0.00 -> 35.5 mm, vias 0 -> 1
- net /Motor3_EN: track 44.6 -> 71.6 mm
- net /Motor2_ENCA: track 42.6 -> 19.4 mm
- net /Motor2_ENCB: track 41.2 -> 18.6 mm
- net /Motor3_M2: track 0.00 -> 20.5 mm, vias 0 -> 1
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- removed copper zone on F.Cu, net +12V
- removed copper zone on F.Cu, net +3.3V
Other:
- board size 92.5 x 92.5 mm -> 80 x 86 mm
- board text removed: "12V"
- board text removed: "3.3V"
- board text removed: "5V"
