File: pcb/omni-wheel/_autosave-omni-wheel.kicad_sch (KiCad schematic)
At the start: 46 parts, among them IC1 AP63301WU-7, IC2 AP63301WU-7, J1 12v TP, J10 Conn_01x01_Pin, J11 Conn_01x01_Pin, J12 5V TP, J13 3.3v TP, J14 GND TP, J15 STLINK, J2 Motor2_output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

Commit message: Added smaller xt connector and power switch
Parts:
- J7: footprint Connector_AMASS:AMASS_XT60PW-M_1x02_P7.20mm_Horizontal -> Connector_AMASS:AMASS_XT30PW-M_1x02_P2.50mm_Horizontal
Changed lines of the file:
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@@
 			)
 		)
-		(property "Footprint" "Connector_AMASS:AMASS_XT60PW-M_1x02_P7.20mm_Horizontal"
+		(property "Footprint" "Connector_AMASS:AMASS_XT30PW-M_1x02_P2.50mm_Horizontal"
 			(at 126.7182 152.9492 0)
 			(effects
